File: PCB/Illuminati.kicad_pcb (KiCad board)
At the start: 2 copper layers, 155 x 79.5 mm, 64 parts, among them J1 Conn_01x17_Socket, J2 USB_C_Receptacle_USB2.0_14P, SW1 SW_Push, SW2 SW_RST, SW3 SW_Push, SW4 SW_Push, SW5 SW_Push, U1 RP2040, U2 W25Q32JVSSIQ_C179173, U3 Radio Module, U4 AP2112K-3.3, U5 USBLC6-2SC6, U6 LIS3DH, X1 X322512MSB4SI

Commit message: firm
Parts:
- added G: LOGO, LOGO, B.Cu at (164.4, 108.9)
- added G***: LOGO, LOGO, B.Cu at (94.6, 105.4)
